Commit message: Renamed descartes_tutorial_puzzle_demo_support to tutorial2_support

File: tutorial2_support/urdf/grinder.xacro (robot description, xacro)
@@ -5,5 +5,5 @@
        <origin xyz="0 0 0" rpy="0 3.14159 0" />
         <geometry>
-          <mesh filename="package://descartes_tutorial_puzzle_demo_support/meshes/grinder_visual.dae" />
+          <mesh filename="package://tutorial2_support/meshes/grinder_visual.dae" />
         </geometry>
       </visual>
@@ -11,5 +11,5 @@
         <origin xyz="0 0 0" rpy="0 3.14159 0" />
         <geometry>
-          <mesh filename="package://descartes_tutorial_puzzle_demo_support/meshes/grinder_collision.dae" />
+          <mesh filename="package://tutorial2_support/meshes/grinder_collision.dae" />
         </geometry>
       </collision>

File: tutorial2_support/urdf/puzzle_mount.xacro (robot description, xacro)
@@ -6,10 +6,10 @@
     <visual>
       <geometry>
-        <mesh filename="package://descartes_tutorial_puzzle_demo_support/meshes/puzzle_mount.stl" />
+        <mesh filename="package://tutorial2_support/meshes/puzzle_mount.stl" />
       </geometry>>
     </visual>
     <collision>
       <geometry>
-        <mesh filename="package://descartes_tutorial_puzzle_demo_support/meshes/puzzle_mount.stl" />
+        <mesh filename="package://tutorial2_support/meshes/puzzle_mount.stl" />
       </geometry>
     </collision>
@@ -30,10 +30,10 @@
     <visual>
       <geometry>
-        <mesh filename="package://descartes_tutorial_puzzle_demo_support/meshes/puzzle_bent.dae" />
+        <mesh filename="package://tutorial2_support/meshes/puzzle_bent.dae" />
       </geometry>
     </visual>
     <collision>
       <geometry>
-        <mesh filename="package://descartes_tutorial_puzzle_demo_support/meshes/puzzle_bent.dae" />
+        <mesh filename="package://tutorial2_support/meshes/puzzle_bent.dae" />
       </geometry>
     </collision>

File: tutorial2_support/urdf/workcell.xacro (robot description, xacro)
@@ -3,6 +3,6 @@
   <xacro:include filename="$(find abb_irb2400_support)/urdf/irb2400_12_155_macro.xacro" />
   <!-- This contains the macro "ses_part_macro" that places the clip wrt the tool tip -->
-  <include filename="$(find descartes_tutorial_puzzle_demo_support)/urdf/puzzle_mount.xacro" />
-  <include filename="$(find descartes_tutorial_puzzle_demo_support)/urdf/grinder.xacro" />
+  <include filename="$(find tutorial2_support)/urdf/puzzle_mount.xacro" />
+  <include filename="$(find tutorial2_support)/urdf/grinder.xacro" />
   <link name="world"/>
   <link name="table">
